File: rcm_noroute.kicad_pcb (KiCad board)
At the start: 2 copper layers, 140 x 70 mm, 159 parts, among them Y1 8MHz, Y2 32.768kHz

Commit message: rcm: apply the GND-to-pour version for review (NOT orderable)
Applied rcm_noroute to rcm.kicad_pcb so it can be looked at. Good board
is in git and at rcm.kicad_pcb.bak_gnd_routed; mfg/ still matches the
GOOD board, not what is on disk.

  good      426/426 routed, 2078 segments, 166 vias, 0 unconnected
  this      293/293 routed, 1605 segments (-23%), 165 vias, 25 unconnected

Electrical DRC is clean on both. What remains here is 8 GND pads the pour
cannot reach - five of them MCU grounds - plus pour-island-to-island
items.

Fixes to stitch_zone_vias.py, all found by running the FULL DRC on the
first attempt rather than only checking connectivity:

  - rescue traces were checked against pads but never against TRACKS, so
    one drove through SR_SCK and shorted it
  - hand-rolled clearance missed hole-to-hole against THT pads; a via
    landed 0.077mm from the battery input
  - stitching was a blanket 4mm grid, 250 vias, most joining the main
    pour to itself for nothing while perforating it

Now stitches only genuine islands (largest filled polygon is the main
pour and is skipped), and validates every placement with the real KiCad
DRC instead of my own arithmetic.

Co-Authored-By: Claude Opus 5 <noreply@anthropic.com>
Routing:
- net GND: track 6.50 -> 5.75 mm, vias 253 -> 40
