File: rcm.kicad_sch (KiCad schematic)
At the start: 155 parts, among them Y1 8MHz, Y2 32.768kHz

Commit message: rcm: FIX D1 wired backwards - board would never have powered up
Diode:SS34 uses KiCad's pin 1 = K, pin 2 = A convention, not the
pin-1-is-anode you would assume. The netlist had D1.1 (cathode) on
+12V_FUSED and D1.2 (anode) on +12V_P, putting the reverse-polarity diode
in backwards. It would have blocked the battery feed outright.

Found by the user reading the schematic symbol and noticing the cathode
bar pointed at the fuse.

Nothing automated caught this and nothing was going to: ERC passes either
orientation because a diode is a valid two-pin connection both ways, and
DRC, the netlist round-trip and the BOM are all equally blind. Same class
as the four faults found in the first schematic review - correct
connectivity, wrong circuit.

Audited the other polarised parts while here; all correct. D_LED1/2 have
anode on pin 2 to the resistor and cathode on pin 1 to GND. D2 works out
right because D_SMA's pad 1 is the cathode and sits on +12V_P - though
Device:D_TVS is a BIDIRECTIONAL symbol standing in for a unidirectional
SMAJ33A, so the schematic cannot express that polarity. Worth swapping
for a directional symbol if revised.

BOTH BOARDS AND BOTH MFG SETS ARE NOW STALE - built from the wrong
circuit, and must be rebuilt and re-routed before anything is ordered.

Co-Authored-By: Claude Opus 5 <noreply@anthropic.com>
Parts:
- JB2: LCSC (none) -> C37208
- J_BOOT: LCSC (none) -> C2937625
- J_SWD: LCSC (none) -> C492404
Connections:
- net +12V_FUSED: now also D1.2 (A); no longer D1.1 (K)
- net +12V_P: now also D1.1 (K); no longer D1.2 (A)
